File: kicad/OPSpec_v0.1.0/OPSpec_v0.1.0.kicad_sch (KiCad schematic)
At the start: 665 parts, among them IC1 PCA9555APW,118, IC2 PCA9555APW,118, IC3 MCP1801T-6002I_OT, IC4 TAR5S50TE85LF, IC5 TAR5S50TE85LF, IC6 TAR5S50TE85LF, IC7 PCA9555APW,118, J1 BASE_INTERFACE, J2 163-179PH-EX, J3 Arduino, J4 TOP_INTERFACE, Q1 NTK3134NT5G, Q10 NTK3134NT5G, Q11 NTK3134NT5G, Q12 NTK3134NT5G, Q13 NXV75UP, Q14 NXV75UP, Q15 NXV75UP, Q16 NXV75UP, Q17 NXV75UP, Q18 NXV75UP, Q19 NXV75UP, Q2 NTK3134NT5G, Q20 NXV75UP, Q21 NXV75UP, Q22 NXV75UP, Q23 NXV75UP, Q24 NXV75UP, Q25 NXV75UP, Q26 NXV75UP, Q27 NXV75UP, Q28 NXV75UP, Q29 NXV75UP, Q3 NTK3134NT5G, Q30 NXV75UP, Q31 NXV75UP, Q32 NXV75UP, Q33 2SCR502UBTL, Q34 2SCR502UBTL, Q35 2SCR502UBTL, Q36 2SCR502UBTL, Q37 2SCR502UBTL, Q38 2SCR502UBTL, Q4 NTK3134NT5G, Q5 NTK3134NT5G, Q6 NTK3134NT5G, Q7 NTK3134NT5G, Q8 NTK3134NT5G, Q9 NTK3134NT5G, T1 S16392-01CT, T10 S16392-01CT, T11 S16392-01CT, T12 S16392-01CT, T13 S16392-01CT, T14 S16392-01CT, T15 S16392-01CT, T16 S16392-01CT, T17 S16392-01CT, T18 S16392-01CT, T19 S16392-01CT, T2 S16392-01CT, T20 S16392-01CT, T21 S16392-01CT, T22 S16392-01CT, T23 S16392-01CT, T24 S16392-01CT, T25 S16392-01CT, T26 S16392-01CT, T27 S16392-01CT, T28 S16392-01CT, T29 S16392-01CT, T3 S16392-01CT, T30 S16392-01CT, T31 S16392-01CT, T32 S16392-01CT, T33 S16392-01CT, T34 S16392-01CT, T35 S16392-01CT, T36 S16392-01CT, T37 S16392-01CT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

Commit message: Prep cleanup
Other:
- note added: "ADC multiplexer 12-bit Address: 1 0 0 1 0 0 0"
- note added: "Address: 0 1 0 0 0 0 0"
- note added: "Address: 0 1 0 0 0 0 1"
- note added: "Address: 0 1 0 0 0 1 1"
- note added: "Address: 0 1 0 0 1 1 1"
- note added: "Total I/O: 12 + 8 LED Switches 12 Detector power grid switches"
- note removed: "ADC multiplexer 12-bit Address: 1 0 0 1 0 0 0 0/1"
- note removed: "Address: 0 1 0 0 0 0 0 0"
- note removed: "Address: 0 1 0 0 0 0 1 0"
- note removed: "Address: 0 1 0 0 0 1 1 0"
- note removed: "Address: 0 1 0 0 1 1 1 0"
- note removed: "Total I/O: 12 + 8 LED Switches 12 Detector signal network switches 12 Detector power grid switches"
Changed lines of the file:
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@@
     (stroke (width 0) (type default) (color 0 0 0 0))
   )
-  (polyline (pts (xy 242.57 297.18) (xy 33.02 297.18))
+  (polyline (pts (xy 242.57 297.18) (xy 31.75 297.18))
     (stroke (width 0) (type default) (color 0 0 0 0))
   )
@@
     (stroke (width 0) (type default) (color 0 0 0 0))
   )
-  (polyline (pts (xy 31.75 193.04) (xy 242.57 191.77))
+  (polyline (pts (xy 31.75 191.77) (xy 242.57 191.77))
     (stroke (width 0) (type default) (color 0 0 0 0))
   )
@@
     (stroke (width 0) (type default) (color 0 0 0 0))
   )
-  (polyline (pts (xy 31.75 193.04) (xy 33.02 297.18))
+  (polyline (pts (xy 31.75 191.77) (xy 31.75 297.18))
     (stroke (width 0) (type default) (color 0 0 0 0))
   )
@@
     )
   )
-  (text "Address: 0 1 0 0 0 0 1 0" (at 177.8 242.57 0)
+  (text "Address: 0 1 0 0 0 0 1" (at 177.8 242.57 0)
     (effects (font (size 1.27 1.27)) (justify left bottom))
   )
-  (text "Address: 0 1 0 0 0 0 0 0" (at 92.71 241.3 0)
+  (text "Address: 0 1 0 0 0 0 0" (at 92.71 241.3 0)
     (effects (font (size 1.27 1.27)) (justify left bottom))
   )
-  (text "Total I/O:\n12 + 8 LED Switches\n12 Detector signal network switches\n12 Detector power grid switches"
+  (text "Total I/O:\n12 + 8 LED Switches\n12 Detector power grid switches"
     (at 491.49 563.88 0)
     (effects (font (size 1.27 1.27)) (justify left bottom))
@@
     (effects (font (size 1.27 1.27)) (justify left bottom))
   )
-  (text "ADC multiplexer 12-bit\n\nAddress:\n1 0 0 1 0 0 0 0/1"
-    (at 547.37 278.13 0)
+  (text "ADC multiplexer 12-bit\n\nAddress:\n1 0 0 1 0 0 0" (at 547.37 278.13 0)
     (effects (font (size 1.27 1.27)) (justify left bottom))
   )
-  (text "Address: 0 1 0 0 0 1 1 0" (at 92.71 290.83 0)
+  (text "Address: 0 1 0 0 0 1 1" (at 92.71 290.83 0)
     (effects (font (size 1.27 1.27)) (justify left bottom))
   )
@@
     (effects (font (size 1.27 1.27)) (justify left bottom))
   )
-  (text "Address: 0 1 0 0 1 1 1 0" (at 179.07 290.83 0)
+  (text "Address: 0 1 0 0 1 1 1" (at 179.07 290.83 0)
     (effects (font (size 1.27 1.27)) (justify left bottom))
   )
@@
   (symbol (lib_id "Mechanical:MountingHole_Pad") (at 675.64 567.69 90) (unit 1)
     (in_bom yes) (on_board yes)
-    (property "Reference" "H3" (id 0) (at 674.37 562.2122 90))
-    (property "Value" "MountingHole" (id 1) (at 674.37 565.15 90))
+    (property "Reference" "H3" (id 0) (at 670.56 566.6541 90))
+    (property "Value" "MountingHole" (id 1) (at 665.48 568.96 90))
     (property "Footprint" "MountingHole:MountingHole_4.3mm_M4_Pad" (id 2) (at 675.64 567.69 0)
       (effects (font (size 1.27 1.27)) hide)
@@
   (symbol (lib_id "Mechanical:MountingHole_Pad") (at 675.64 574.04 90) (unit 1)
     (in_bom yes) (on_board yes)
-    (property "Reference" "H4" (id 0) (at 674.37 568.5622 90))
-    (property "Value" "MountingHole" (id 1) (at 674.37 571.5 90))
+    (property "Reference" "H4" (id 0) (at 670.56 573.0041 90))
+    (property "Value" "MountingHole" (id 1) (at 665.48 575.31 90))
     (property "Footprint" "MountingHole:MountingHole_4.3mm_M4_Pad" (id 2) (at 675.64 574.04 0)
       (effects (font (size 1.27 1.27)) hide)
@@
   (symbol (lib_id "Mechanical:MountingHole_Pad") (at 675.64 554.99 90) (unit 1)
     (in_bom yes) (on_board yes)
-    (property "Reference" "H1" (id 0) (at 674.37 549.9131 90))
-    (property "Value" "MountingHole" (id 1) (at 674.37 552.45 90))
+    (property "Reference" "H1" (id 0) (at 670.56 554.355 90))
+    (property "Value" "MountingHole" (id 1) (at 665.48 556.26 90))
     (property "Footprint" "MountingHole:MountingHole_4.3mm_M4_Pad" (id 2) (at 675.64 554.99 0)
       (effects (font (size 1.27 1.27)) hide)
@@
   (symbol (lib_id "Mechanical:MountingHole_Pad") (at 675.64 561.34 90) (unit 1)
     (in_bom yes) (on_board yes)
-    (property "Reference" "H2" (id 0) (at 674.37 555.8622 90))
-    (property "Value" "MountingHole" (id 1) (at 674.37 558.8 90))
+    (property "Reference" "H2" (id 0) (at 670.56 560.3041 90))
+    (property "Value" "MountingHole" (id 1) (at 665.48 562.61 90))
     (property "Footprint" "MountingHole:MountingHole_4.3mm_M4_Pad" (id 2) (at 675.64 561.34 0)
       (effects (font (size 1.27 1.27)) hide)
